File: Current_Sensor.kicad_sch (KiCad schematic)
At the start: 6 parts

Commit message: Тестовая версия
Parts:
- removed C29: 2.2u, Capacitor_SMD:C_0805_2012Metric_Pad1.18x1.45mm_HandSolder, symbol Device:C_Small
- removed D18: ADM3485E, Package_SO:SOIC-8_3.9x4.9mm_P1.27mm, symbol Interface_My:ADM3485E
- removed R24: 120, Resistor_SMD:R_0805_2012Metric_Pad1.20x1.40mm_HandSolder, symbol Device:R_Small
Connections:
- net Current: now reaches C28.1, D17.12 (VOUT)
- net E3 renamed OUT2
- net OUT+ renamed OUT2_Sens
- no-connect marks 2 -> 1

Commit message: Развел все дорожки
Connections:
- net OUT2: now also D17.5 (IP-), D17.6 (IP-), D17.7 (IP-), D17.8 (IP-); no longer D17.1 (IP+), D17.2 (IP+), D17.3 (IP+), D17.4 (IP+)
- net OUT2_Sens: now also D17.1 (IP+), D17.2 (IP+), D17.3 (IP+), D17.4 (IP+); no longer D17.5 (IP-), D17.6 (IP-), D17.7 (IP-), D17.8 (IP-)
Other:
- moved on the sheet: C27, C28
