File: Indication.kicad_sch (KiCad schematic)
At the start: 13 parts

Commit message: VER2.1: исправил BOM, наименования в схеме и добавил папку с документами
Parts:
- D14: value ADM1485JRZ -> SN65HVD3082EDR
Changed lines of the file:
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@@
 			)
 		)
-		(property "Description" "FYLS-0805UBC"
+		(property "Description" "LTST-C171TBKT"
 			(at 76.2 136.398 0)
 			(effects
@@
 			)
 		)
-		(property "Description" "KP-2012SURCK"
+		(property "Description" "EC04-0805QRC/E-AV"
 			(at 76.2 111.76 0)
 			(effects
@@
 			)
 		)
-		(property "Value" "ADM1485JRZ"
+		(property "Value" "SN65HVD3082EDR"
 			(at 231.648 91.44 0)
 			(effects
