File: Driver_Inductor.kicad_pcb (KiCad board)
At the start: 6 copper layers, 119.6 x 60.5 mm, 99 parts, among them J1 Control_A, J2 DC+, J3 DC-, J4 OUT1, J5 OUT2, Q1 BC817, U3 LM1117GS-5.0, U4 LMV7219M5, U5 ADuM1200AR

Commit message: VER2.1: добавил файлы для сборки платы
Parts:
- J2: value DC+ -> J2
- J3: value DC- -> J3
- J4: value OUT1 -> J4
- J5: value OUT2 -> J5
