File: Driver_Inductor.kicad_sch (KiCad schematic)
At the start: 104 parts, among them J1 Control_A, J2 DC+, J3 DC-, J4 OUT1, J5 OUT2, Q1 BC817, U3 LM1117GS-5.0, U4 LMV7219M5, U5 SCM3728ASA

Commit message: VER2.2: создал папку для производственных доков
Parts:
- C1, C11, C12, C13, C15, C16, C2, C27, C28, C3, C30, C31, C32, C33, C34, C35, C36, C4, C5, C6, C7, C8, C9: Description P/N (none) -> Capacitor SMD 25+V
- C10: Description P/N (none) -> Capacitor 630V
- C14, C19, C21, C29, C37: Description P/N (none) -> Capacitor SMD 630V
- C17, C18, C20, C22, C23, C24, C25, C26: Description P/N (none) -> Capacitor SMD 50+V
- D1, D2: value NSI6651ASC-DSWR -> ~; Description P/N (none) -> Gate Driver; Product Name (none) -> NSI6651ASC-DSWR
- D10: value RDY -> ~; Description P/N (none) -> Blue LED; Product Name (none) -> FYLS-0805UBC; Purpose (none) -> RDY
- D11, D8: value WRA1215S-3WR2 -> ~; Description P/N (none) -> DCDC; Product Name (none) -> WRA1215S-3WR2
- D12: value K7805M-1000R3 -> ~; Description P/N (none) -> DCDC; Product Name (none) -> K7805M-1000R3
- D13, D14, D15: value SN65HVD3082EDR -> ~; Description P/N (none) -> RS485; Product Name (none) -> SN65HVD3082EDR
- D16, D18: value 1SMB5919B -> ~; Description P/N (none) -> Zener Diode; Product Name (none) -> 1SMB5919B
- D17: value NSM2011-50B5R-DSWR -> ~; Description P/N (none) -> Current Sensor; Product Name (none) -> NSM2011-50B5R-DSWR
- D19: value ADM3485E -> ~; Description P/N (none) -> RS485; Product Name (none) -> SN65HVD3082EDR
- D20: value GD50FFY120C5S -> ~; Description P/N (none) -> IGBT Module; Product Name (none) -> GD50FFY120C5S
- D3, D4: value MMSZ5240B -> ~; Description P/N (none) -> Zener Diode; Product Name (none) -> MMSZ5240B
- D5, D7: value MURS160 -> ~; Description P/N (none) -> Diode; Product Name (none) -> MURS160
- D6: value SN74AHC1G08DBVR -> ~; Description P/N (none) -> AND; Product Name (none) -> SN74AHC1G08DBVR
- D9: value FLT -> ~; Description P/N (none) -> Red LED; Product Name (none) -> FYLS-0805URC; Purpose (none) -> FLT
- J1: value Control_A -> ~; Description P/N (none) -> Connector; Product Name (none) -> SCT3001WV-2x06P; Purpose (none) -> Control_A
- J2: value DC+ -> ~; Description P/N (none) -> Connector; Product Name (none) -> M4 Bush SMD; Purpose (none) -> DC+
- J3: value DC- -> ~; Description P/N (none) -> Connector; Product Name (none) -> M4 Bush SMD; Purpose (none) -> DC-
- J4: value OUT1 -> ~; Description P/N (none) -> Connector; Product Name (none) -> M4 Bush SMD; Purpose (none) -> OUT1
- J5: value OUT2 -> ~; Description P/N (none) -> Connector; Product Name (none) -> M4 Bush SMD; Purpose (none) -> OUT2
- Q1: value BC817 -> ~; Description P/N (none) -> MOSFET; Product Name (none) -> BC817
- R1, R10, R11, R12, R13, R14, R15, R16, R17, R18, R19, R2, R20, R21, R22, R23, R24, R25, R26, R27, R28, R29, R3, R30, R31, R32, R33, R34, R35, R36, R37, R38, R4, R5, R6, R7, R8, R9: Description P/N (none) -> Resistor SMD
- U3: value LM1117GS-5.0 -> ~; Description P/N (none) -> Linear Regulator; Product Name (none) -> LM1117GS-5.0
- U4: value LMV7219M5 -> ~; Description P/N (none) -> Comparator; Product Name (none) -> LMV7219M5
- U5: value SCM3728ASA -> ~; Description P/N (none) -> Digital Isolator; Product Name (none) -> SCM3728ASA
